File: PCB/EKR82_Pro.kicad_pcb (KiCad board)
At the start: 2 copper layers, 173 x 137 mm, 99 parts, among them J1 LED, J2 4PIN, P1 i2c_pin, P2 i2c_pin, SW1 SW_PUSH, SW10 SW_PUSH, SW11 SW_PUSH, SW12 SW_PUSH, SW13 SW_PUSH, SW14 SW_PUSH, SW15 SW_PUSH, SW16 SW_PUSH, SW17 SW_PUSH, SW18 SW_PUSH, SW19 SW_PUSH, SW2 SW_PUSH, SW20 SW_PUSH, SW21 SW_PUSH, SW22 SW_PUSH, SW23 SW_PUSH, SW24 SW_PUSH, SW25 SW_PUSH, SW26 SW_PUSH, SW27 SW_PUSH, SW28 SW_PUSH, SW29 SW_PUSH, SW3 SW_PUSH, SW30 SW_PUSH, SW31 SW_PUSH, SW32 SW_PUSH, SW33 SW_PUSH, SW34 SW_PUSH, SW35 SW_PUSH, SW36 SW_PUSH, SW37 SW_PUSH, SW38 SW_PUSH, SW39 SW_PUSH, SW4 SW_PUSH, SW40 SW_PUSH, SW41 SW_PUSH, SW5 SW_PUSH, SW6 SW_PUSH, SW7 SW_PUSH, SW8 SW_PUSH, SW9 SW_PUSH, U1 ProMicro

Commit message: change name lily58 to EKR82
Parts:
- D10, D11, D12, D13, D14, D15, D16, D17, D18, D19, D20, D21, D22, D23, D24, D5, D6, D7, D8, D9: footprint Lily58-footprint:Diode_SOD123 -> EKR82-footprint:Diode_SOD123
- J1: footprint Lily58-footprint:LED -> EKR82-footprint:LED
- J2: footprint Lily58-footprint:MJ-4PP-9 -> EKR82-footprint:MJ-4PP-9
- P1, P2: footprint Lily58-footprint:1pin_conn -> EKR82-footprint:1pin_conn
- R1, R2: footprint Lily58-footprint:RESISTOR_mini -> EKR82-footprint:RESISTOR_mini
- RSW1: footprint Lily58-footprint:TACT_SWITCH_TVBP06 -> EKR82-footprint:TACT_SWITCH_TVBP06
- TH3, TH4, TH5, TH6, TH7: footprint Lily58-footprint:HOLE_M2_TH -> EKR82-footprint:HOLE_M2_TH
- U1: footprint Lily58-footprint:ProMicro_rev2 -> EKR82-footprint:ProMicro_rev2
- W1: footprint Lily58-footprint:jumper_data -> EKR82-footprint:jumper_data
Changed lines of the file:
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@@
       (net 41 col5))
   )
-  (module Lily58-footprint:MJ-4PP-9 (layer F.Cu)
+  (module EKR82-footprint:MJ-4PP-9 (layer F.Cu)
     (at 87.9 39.3)
     (fp_text reference J2 (at -0.1 15.1) (layer F.SilkS) hide
@@
     )
   )
-  (module Lily58-footprint:LED (layer F.Cu)
+  (module EKR82-footprint:LED (layer F.Cu)
     (at 112.7 81.1 180)
     (fp_text reference J1 (at 0 -2.54 180) (layer F.SilkS) hide
@@
       (net 34 VCC))
   )
-  (module Lily58-footprint:ProMicro_rev2 (layer F.Cu)
+  (module EKR82-footprint:ProMicro_rev2 (layer F.Cu)
     (at 101 56)
     (fp_text reference U1 (at 0 1.2) (layer F.SilkS) hide
@@
       (net 45 RESET))
   )
-  (module Lily58-footprint:HOLE_M2_TH (layer F.Cu)
+  (module EKR82-footprint:HOLE_M2_TH (layer F.Cu)
     (at 129.6 59.6)
     (fp_text reference TH3 (at 0 -2.54) (layer F.SilkS) hide
@@
       (clearance 0.3))
   )
-  (module Lily58-footprint:HOLE_M2_TH (layer F.Cu)
+  (module EKR82-footprint:HOLE_M2_TH (layer F.Cu)
     (at 205.8 61.8)
     (fp_text reference TH4 (at 0 -2.54) (layer F.SilkS) hide
@@
       (clearance 0.3))
   )
-  (module Lily58-footprint:HOLE_M2_TH (layer F.Cu)
+  (module EKR82-footprint:HOLE_M2_TH (layer F.Cu)
     (at 129.6 97.6)
     (fp_text reference TH5 (at 0 -2.54) (layer F.SilkS) hide
@@
       (clearance 0.3))
   )
-  (module Lily58-footprint:HOLE_M2_TH (layer F.Cu)
+  (module EKR82-footprint:HOLE_M2_TH (layer F.Cu)
     (at 224.8 100)
     (fp_text reference TH6 (at 0 -2.54) (layer F.SilkS) hide
@@
       (clearance 0.3))
   )
-  (module Lily58-footprint:HOLE_M2_TH (layer F.Cu)
+  (module EKR82-footprint:HOLE_M2_TH (layer F.Cu)
     (at 94.615 117.475 90)
     (fp_text reference TH7 (at 0 -2.54 90) (layer F.SilkS) hide
@@
       (clearance 0.3))
   )
-  (module Lily58-footprint:1pin_conn (layer F.Cu)
+  (module EKR82-footprint:1pin_conn (layer F.Cu)
     (at 84.7 60.7 180)
     (descr "Resitance 3 pas")
@@
     )
   )
-  (module Lily58-footprint:1pin_conn (layer F.Cu)
+  (module EKR82-footprint:1pin_conn (layer F.Cu)
     (at 86.9 60.7 180)
     (descr "Resitance 3 pas")
@@
     )
   )
-  (module Lily58-footprint:RESISTOR_mini (layer F.Cu)
+  (module EKR82-footprint:RESISTOR_mini (layer F.Cu)
     (at 86.938035 56.039272 270)
     (descr "Resitance 3 pas")
@@
     )
   )
-  (module Lily58-footprint:RESISTOR_mini (layer F.Cu)
+  (module EKR82-footprint:RESISTOR_mini (layer F.Cu)
     (at 84.688035 56.039272 270)
     (descr "Resitance 3 pas")
@@
     )
   )
-  (module Lily58-footprint:TACT_SWITCH_TVBP06 (layer F.Cu)
+  (module EKR82-footprint:TACT_SWITCH_TVBP06 (layer F.Cu)
     (at 85 67.7 90)
     (fp_text reference RSW1 (at 0 -1.7 90) (layer F.SilkS) hide
@@
       (net 45 RESET))
   )
-  (module Lily58-footprint:jumper_data (layer F.Cu)
+  (module EKR82-footprint:jumper_data (layer F.Cu)
     (at 89 60.7 90)
     (attr smd)
@@
     )
   )
-  (module Lily58-footprint:Diode_SOD123 placed (layer F.Cu)
+  (module EKR82-footprint:Diode_SOD123 placed (layer F.Cu)
     (at 190.6 60.4)
     (descr "Diode, DO-41, SOD81, Horizontal, RM 10mm,")
@@
       (net 5 row0))
   )
-  (module Lily58-footprint:Diode_SOD123 placed (layer F.Cu)
+  (module EKR82-footprint:Diode_SOD123 placed (layer F.Cu)
     (at 221.8 61.8)
     (descr "Diode, DO-41, SOD81, Horizontal, RM 10mm,")
@@
       (net 10 "Net-(D6-Pad2)"))
   )
-  (module Lily58-footprint:Diode_SOD123 placed (layer F.Cu)
+  (module EKR82-footprint:Diode_SOD123 placed (layer F.Cu)
     (at 114.4 61.1)
     (descr "Diode, DO-41, SOD81, Horizontal, RM 10mm,")
@@
       (net 7 row1))
   )
-  (module Lily58-footprint:Diode_SOD123 placed (layer F.Cu)
+  (module EKR82-footprint:Diode_SOD123 placed (layer F.Cu)
     (at 135.3 58.7)
     (descr "Diode, DO-41, SOD81, Horizontal, RM 10mm,")
@@
       (net 7 row1))
   )
-  (module Lily58-footprint:Diode_SOD123 placed (layer F.Cu)
+  (module EKR82-footprint:Diode_SOD123 placed (layer F.Cu)
     (at 152.6 57.4)
     (descr "Diode, DO-41, SOD81, Horizontal, RM 10mm,")
@@
       (net 7 row1))
   )
-  (module Lily58-footprint:Diode_SOD123 placed (layer F.Cu)
+  (module EKR82-footprint:Diode_SOD123 placed (layer F.Cu)
     (at 171.5 58.7)
     (descr "Diode, DO-41, SOD81, Horizontal, RM 10mm,")
@@
       (net 15 "Net-(D10-Pad2)"))
   )
-  (module Lily58-footprint:Diode_SOD123 placed (layer F.Cu)
+  (module EKR82-footprint:Diode_SOD123 placed (layer F.Cu)
     (at 190.6 63.3)
     (descr "Diode, DO-41, SOD81, Horizontal, RM 10mm,")
@@
       (net 7 row1))
   )
-  (module Lily58-footprint:Diode_SOD123 placed (layer F.Cu)
+  (module EKR82-footprint:Diode_SOD123 placed (layer F.Cu)
     (at 221.8 64.9)
     (descr "Diode, DO-41, SOD81, Horizontal, RM 10mm,")
@@
       (net 7 row1))
   )
-  (module Lily58-footprint:Diode_SOD123 placed (layer F.Cu)
+  (module EKR82-footprint:Diode_SOD123 placed (layer F.Cu)
     (at 114.4 96)
     (descr "Diode, DO-41, SOD81, Horizontal, RM 10mm,")
@@
       (net 18 "Net-(D13-Pad2)"))
   )
-  (module Lily58-footprint:Diode_SOD123 placed (layer F.Cu)
+  (module EKR82-footprint:Diode_SOD123 placed (layer F.Cu)
     (at 134.3 93.8)
     (descr "Diode, DO-41, SOD81, Horizontal, RM 10mm,")
@@
       (net 9 row2))
   )
-  (module Lily58-footprint:Diode_SOD123 placed (layer F.Cu)
+  (module EKR82-footprint:Diode_SOD123 placed (layer F.Cu)
     (at 152.5 92.3)
     (descr "Diode, DO-41, SOD81, Horizontal, RM 10mm,")
@@
       (net 9 row2))
   )
-  (module Lily58-footprint:Diode_SOD123 placed (layer F.Cu)
+  (module EKR82-footprint:Diode_SOD123 placed (layer F.Cu)
     (at 171.5 93.6)
     (descr "Diode, DO-41, SOD81, Horizontal, RM 10mm,")
@@
       (net 21 "Net-(D16-Pad2)"))
   )
-  (module Lily58-footprint:Diode_SOD123 placed (layer F.Cu)
+  (module EKR82-footprint:Diode_SOD123 placed (layer F.Cu)
     (at 190.6 98.3)
     (descr "Diode, DO-41, SOD81, Horizontal, RM 10mm,")
@@
       (net 22 "Net-(D17-Pad2)"))
   )
-  (module Lily58-footprint:Diode_SOD123 placed (layer F.Cu)
+  (module EKR82-footprint:Diode_SOD123 placed (layer F.Cu)
     (at 215.61 96.99)
     (descr "Diode, DO-41, SOD81, Horizontal, RM 10mm,")
@@
       (net 9 row2))
   )
-  (module Lily58-footprint:Diode_SOD123 placed (layer F.Cu)
+  (module EKR82-footprint:Diode_SOD123 placed (layer F.Cu)
     (at 114.4 99.1)
     (descr "Diode, DO-41, SOD81, Horizontal, RM 10mm,")
@@
       (net 11 row3))
   )
-  (module Lily58-footprint:Diode_SOD123 placed (layer F.Cu)
+  (module EKR82-footprint:Diode_SOD123 placed (layer F.Cu)
     (at 135.3 96.8)
     (descr "Diode, DO-41, SOD81, Horizontal, RM 10mm,")
@@
       (net 25 "Net-(D20-Pad2)"))
   )
-  (module Lily58-footprint:Diode_SOD123 placed (layer F.Cu)
+  (module EKR82-footprint:Diode_SOD123 placed (layer F.Cu)
     (at 152.5 95.4)
     (descr "Diode, DO-41, SOD81, Horizontal, RM 10mm,")
@@
       (net 11 row3))
   )
-  (module Lily58-footprint:Diode_SOD123 placed (layer F.Cu)
+  (module EKR82-footprint:Diode_SOD123 placed (layer F.Cu)
     (at 171.5 96.8)
     (descr "Diode, DO-41, SOD81, Horizontal, RM 10mm,")
@@
       (net 27 "Net-(D22-Pad2)"))
   )
-  (module Lily58-footprint:Diode_SOD123 placed (layer F.Cu)
+  (module EKR82-footprint:Diode_SOD123 placed (layer F.Cu)
     (at 190.6 101.5)
     (descr "Diode, DO-41, SOD81, Horizontal, RM 10mm,")
@@
       (net 11 row3))
   )
-  (module Lily58-footprint:Diode_SOD123 placed (layer F.Cu)
+  (module EKR82-footprint:Diode_SOD123 placed (layer F.Cu)
     (at 215.94 102.32)
     (descr "Diode, DO-41, SOD81, Horizontal, RM 10mm,")
