File: PCB/EKR82_Pro.sch (KiCad schematic (older format))
At the start: 95 parts, among them J1 LED, J2 4PIN, P1 i2c_pin, P2 i2c_pin, SW1 SW_PUSH, SW10 SW_PUSH, SW11 SW_PUSH, SW12 SW_PUSH, SW13 SW_PUSH, SW14 SW_PUSH, SW15 SW_PUSH, SW16 SW_PUSH, SW17 SW_PUSH, SW18 SW_PUSH, SW19 SW_PUSH, SW2 SW_PUSH, SW20 SW_PUSH, SW21 SW_PUSH, SW22 SW_PUSH, SW23 SW_PUSH, SW24 SW_PUSH, SW25 SW_PUSH, SW26 SW_PUSH, SW27 SW_PUSH, SW28 SW_PUSH, SW29 SW_PUSH, SW3 SW_PUSH, SW30 SW_PUSH, SW31 SW_PUSH, SW32 SW_PUSH, SW33 SW_PUSH, SW34 SW_PUSH, SW35 SW_PUSH, SW36 SW_PUSH, SW37 SW_PUSH, SW38 SW_PUSH, SW39 SW_PUSH, SW4 SW_PUSH, SW40 SW_PUSH, SW5 SW_PUSH, SW6 SW_PUSH, SW7 SW_PUSH, SW8 SW_PUSH, SW9 SW_PUSH, U1 ProMicro

Commit message: change name lily58 to EKR82
Parts:
- added D41: D, keyboard_switch:Diode_SOD123, symbol EKR82_Pro-rescue:D-EKR82-cache
- added SW41: SW_PUSH, keyboard_switch:CherryMX_KailhLowProfile_Hotswap_edge-2, symbol EKR82_Pro-rescue:SW_PUSH-EKR82-cache
- D1, D2, D25, D26, D27, D28, D29, D3, D30, D31, D32, D33, D34, D35, D36, D37, D38, D39, D4, D40: symbol Lily58_Pro-rescue:D-Lily58-cache -> EKR82_Pro-rescue:D-EKR82-cache
- D10, D11, D12, D13, D14, D15, D16, D17, D18, D19, D20, D21, D22, D23, D24, D5, D6, D7, D8, D9: footprint Lily58-footprint:Diode_SOD123 -> EKR82-footprint:Diode_SOD123; symbol Lily58_Pro-rescue:D-Lily58-cache -> EKR82_Pro-rescue:D-EKR82-cache
- J1: footprint Lily58-footprint:LED -> EKR82-footprint:LED; symbol Lily58_Pro-rescue:LED-Lily58-cache -> EKR82_Pro-rescue:LED-EKR82-cache
- J2: footprint Lily58-footprint:MJ-4PP-9 -> EKR82-footprint:MJ-4PP-9; symbol Lily58_Pro-rescue:MJ-4PP-9-Lily58-cache -> EKR82_Pro-rescue:MJ-4PP-9-EKR82-cache
- P1, P2: footprint Lily58-footprint:1pin_conn -> EKR82-footprint:1pin_conn; symbol Lily58_Pro-rescue:i2c_pin-Lily58-cache -> EKR82_Pro-rescue:i2c_pin-EKR82-cache
- R1, R2: footprint Lily58-footprint:RESISTOR_mini -> EKR82-footprint:RESISTOR_mini; symbol Lily58_Pro-rescue:R-Lily58-cache -> EKR82_Pro-rescue:R-EKR82-cache
- RSW1: footprint Lily58-footprint:TACT_SWITCH_TVBP06 -> EKR82-footprint:TACT_SWITCH_TVBP06; symbol Lily58_Pro-rescue:SW_RST-Lily58-cache -> EKR82_Pro-rescue:SW_RST-EKR82-cache
- SW1, SW10, SW11, SW12, SW13, SW14, SW15, SW16, SW17, SW18, SW19, SW2, SW20, SW21, SW22, SW23, SW24, SW25, SW26, SW27, SW28, SW29, SW3, SW30, SW31, SW32, SW33, SW34, SW35, SW36, SW37, SW38, SW39, SW4, SW40, SW5, SW6, SW7, SW8, SW9: symbol Lily58_Pro-rescue:SW_PUSH-Lily58-cache -> EKR82_Pro-rescue:SW_PUSH-EKR82-cache
- TH3, TH4, TH5, TH6, TH7: footprint Lily58-footprint:HOLE_M2_TH -> EKR82-footprint:HOLE_M2_TH; symbol Lily58_Pro-rescue:HOLE-Lily58-cache -> EKR82_Pro-rescue:HOLE-EKR82-cache
- TH8: symbol Lily58_Pro-rescue:HOLE-Lily58-cache -> EKR82_Pro-rescue:HOLE-EKR82-cache
- U1: footprint Lily58-footprint:ProMicro_rev2 -> EKR82-footprint:ProMicro_rev2; symbol Lily58_Pro-rescue:ProMicro_2-Lily58-cache -> EKR82_Pro-rescue:ProMicro_2-EKR82-cache
- W1: footprint Lily58-footprint:jumper_data -> EKR82-footprint:jumper_data
Connections:
- wire segments 83 -> 85
