File: PCB/EKR82.sch (KiCad schematic (older format))
At the start: 97 parts, among them J1 LED, J2 4PIN, P1 i2c_pin, P2 i2c_pin, SW1 SW_PUSH, SW10 SW_PUSH, SW11 SW_PUSH, SW12 SW_PUSH, SW13 SW_PUSH, SW14 SW_PUSH, SW15 SW_PUSH, SW16 SW_PUSH, SW17 SW_PUSH, SW18 SW_PUSH, SW19 SW_PUSH, SW2 SW_PUSH, SW20 SW_PUSH, SW21 SW_PUSH, SW22 SW_PUSH, SW23 SW_PUSH, SW24 SW_PUSH, SW25 SW_PUSH, SW26 SW_PUSH, SW27 SW_PUSH, SW28 SW_PUSH, SW29 SW_PUSH, SW3 SW_PUSH, SW30 SW_PUSH, SW31 SW_PUSH, SW32 SW_PUSH, SW33 SW_PUSH, SW34 SW_PUSH, SW35 SW_PUSH, SW36 SW_PUSH, SW37 SW_PUSH, SW38 SW_PUSH, SW39 SW_PUSH, SW4 SW_PUSH, SW40 SW_PUSH, SW41 SW_PUSH, SW5 SW_PUSH, SW6 SW_PUSH, SW7 SW_PUSH, SW8 SW_PUSH, SW9 SW_PUSH, U1 ProMicro

Commit message: rename kicad project EKR82_Pro to EKR82
Parts:
- D1, D10, D11, D12, D13, D14, D15, D16, D17, D18, D19, D2, D20, D21, D22, D23, D24, D25, D26, D27, D28, D29, D3, D30, D31, D32, D33, D34, D35, D36, D37, D38, D39, D4, D40, D41, D5, D6, D7, D8, D9: symbol EKR82_Pro-rescue:D-EKR82-cache -> EKR82-rescue:D-EKR82-cache
- J1: symbol EKR82_Pro-rescue:LED-EKR82-cache -> EKR82-rescue:LED-EKR82-cache
- J2: symbol EKR82_Pro-rescue:MJ-4PP-9-EKR82-cache -> EKR82-rescue:MJ-4PP-9-EKR82-cache
- P1, P2: symbol EKR82_Pro-rescue:i2c_pin-EKR82-cache -> EKR82-rescue:i2c_pin-EKR82-cache
- R1, R2: symbol EKR82_Pro-rescue:R-EKR82-cache -> EKR82-rescue:R-EKR82-cache
- RSW1: symbol EKR82_Pro-rescue:SW_RST-EKR82-cache -> EKR82-rescue:SW_RST-EKR82-cache
- SW1, SW10, SW11, SW12, SW13, SW14, SW15, SW16, SW17, SW18, SW19, SW2, SW20, SW21, SW22, SW23, SW24, SW25, SW26, SW27, SW28, SW29, SW3, SW30, SW31, SW32, SW33, SW34, SW35, SW36, SW37, SW38, SW39, SW4, SW40, SW41, SW5, SW6, SW7, SW8, SW9: symbol EKR82_Pro-rescue:SW_PUSH-EKR82-cache -> EKR82-rescue:SW_PUSH-EKR82-cache
- TH3, TH4, TH5, TH6, TH7, TH8: symbol EKR82_Pro-rescue:HOLE-EKR82-cache -> EKR82-rescue:HOLE-EKR82-cache
- U1: symbol EKR82_Pro-rescue:ProMicro_2-EKR82-cache -> EKR82-rescue:ProMicro_2-EKR82-cache

Commit message: move SW41 and remove resistors
Parts:
- removed R1, R2: R, EKR82-footprint:RESISTOR_mini, symbol EKR82-rescue:R-EKR82-cache
- removed W1: jumper, EKR82-footprint:jumper_data, symbol Device:Jumper

Commit message: add backlight rgb WIP
Parts:
- added D42, D43, D44, D45, D46, D47, D48, D49, D50, D51, D52, D53, D54, D55, D56, D57, D58, D59, D60, D61, D62, D63: SK6812MINI, LED_SMD:LED_SK6812MINI_PLCC4_3.5x3.5mm_P1.75mm, symbol LED:SK6812MINI
- added P3: led1, Connector_PinHeader_1.27mm:PinHeader_1x01_P1.27mm_Vertical, symbol EKR82-rescue:i2c_pin-EKR82-cache
Connections:
- wire segments 85 -> 130

Commit message: add led and logo
Parts:
- added THLogo1: HOLE, EKR82-footprint:EKR82-2, symbol EKR82-rescue:HOLE-EKR82-cache
- added THLogo2, THLogo3: HOLE, Symbol:OSHW-Symbol_8.9x8mm_SilkScreen, symbol EKR82-rescue:HOLE-EKR82-cache
- D42, D43, D44, D45, D46, D47, D48, D49, D50, D51, D52, D53, D54, D55, D56, D57, D58, D59, D60, D61, D62, D63: symbol LED:SK6812MINI -> EKR82-rescue:SK6812MINI-LED
Changed lines of the file:
@@
 $EndComp
 $Comp
-L LED:SK6812MINI D43
+L EKR82-rescue:SK6812MINI-LED D43
 U 1 1 60C19178
 P 3100 9450
@@
 $EndComp
 $Comp
-L LED:SK6812MINI D44
+L EKR82-rescue:SK6812MINI-LED D44
 U 1 1 60C1D7C9
 P 3700 9450
@@
 $EndComp
 $Comp
-L LED:SK6812MINI D45
+L EKR82-rescue:SK6812MINI-LED D45
 U 1 1 60C1D7CF
 P 4300 9450
@@
 $EndComp
 $Comp
-L LED:SK6812MINI D46
+L EKR82-rescue:SK6812MINI-LED D46
 U 1 1 60C24290
 P 4900 9450
@@
 $EndComp
 $Comp
-L LED:SK6812MINI D47
+L EKR82-rescue:SK6812MINI-LED D47
 U 1 1 60C24296
 P 5500 9450
@@
 $EndComp
 $Comp
-L LED:SK6812MINI D48
+L EKR82-rescue:SK6812MINI-LED D48
 U 1 1 60C2429C
 P 6100 9450
@@
 $EndComp
 $Comp
-L LED:SK6812MINI D49
+L EKR82-rescue:SK6812MINI-LED D49
 U 1 1 60C242A2
 P 6700 9450
@@
 $EndComp
 $Comp
-L LED:SK6812MINI D50
+L EKR82-rescue:SK6812MINI-LED D50
 U 1 1 60C292EA
 P 7300 9450
@@
 $EndComp
 $Comp
-L LED:SK6812MINI D51
+L EKR82-rescue:SK6812MINI-LED D51
 U 1 1 60C292F0
 P 7900 9450
@@
 $EndComp
 $Comp
-L LED:SK6812MINI D52
+L EKR82-rescue:SK6812MINI-LED D52
 U 1 1 60C292F6
 P 1900 9450
@@
 	7900 9750 8500 9750
 $Comp
-L power:VCC #PWR0103
+L EKR82-rescue:VCC-power #PWR0103
 U 1 1 60C31362
 P 2500 9750
@@
 $EndComp
 $Comp
-L power:GND #PWR0104
+L EKR82-rescue:GND-power #PWR0104
 U 1 1 60C3AF7B
 P 2500 9150
@@
 Connection ~ 2500 9150
 $Comp
-L LED:SK6812MINI D42
+L EKR82-rescue:SK6812MINI-LED D42
 U 1 1 60C12BC0
 P 2500 9450
@@
 	2500 9750 1900 9750
 $Comp
-L LED:SK6812MINI D55
+L EKR82-rescue:SK6812MINI-LED D55
 U 1 1 60CA85DF
 P 3100 8350
@@
 $EndComp
 $Comp
-L LED:SK6812MINI D56
+L EKR82-rescue:SK6812MINI-LED D56
 U 1 1 60CA85E5
 P 3700 8350
@@
 $EndComp
 $Comp
-L LED:SK6812MINI D57
+L EKR82-rescue:SK6812MINI-LED D57
 U 1 1 60CA85EB
 P 4300 8350
@@
 $EndComp
 $Comp
-L LED:SK6812MINI D58
+L EKR82-rescue:SK6812MINI-LED D58
 U 1 1 60CA85F1
 P 4900 8350
@@
 $EndComp
 $Comp
-L LED:SK6812MINI D59
+L EKR82-rescue:SK6812MINI-LED D59
 U 1 1 60CA85F7
 P 5500 8350
@@
 $EndComp
 $Comp
-L LED:SK6812MINI D60
+L EKR82-rescue:SK6812MINI-LED D60
 U 1 1 60CA85FD
 P 6100 8350
@@
 $EndComp
 $Comp
-L LED:SK6812MINI D61
+L EKR82-rescue:SK6812MINI-LED D61
 U 1 1 60CA8603
 P 6700 8350
@@
 $EndComp
 $Comp
-L LED:SK6812MINI D62
+L EKR82-rescue:SK6812MINI-LED D62
 U 1 1 60CA8609
 P 7300 8350
@@
 $EndComp
 $Comp
-L LED:SK6812MINI D63
+L EKR82-rescue:SK6812MINI-LED D63
 U 1 1 60CA860F
 P 7900 8350
@@
 $EndComp
 $Comp
-L LED:SK6812MINI D53
+L EKR82-rescue:SK6812MINI-LED D53
 U 1 1 60CA8615
 P 1900 8350
@@
 	7900 8650 8500 8650
 $Comp
-L power:VCC #PWR0105
+L EKR82-rescue:VCC-power #PWR0105
 U 1 1 60CA8641
 P 2500 8650
@@
 $EndComp
 $Comp
-L power:GND #PWR0106
+L EKR82-rescue:GND-power #PWR0106
 U 1 1 60CA8647
 P 2500 8050
@@
 Connection ~ 2500 8050
 $Comp
-L LED:SK6812MINI D54
+L EKR82-rescue:SK6812MINI-LED D54
 U 1 1 60CA864F
 P 2500 8350
@@
 	1600 9450 1600 8350
 Connection ~ 1600 9450
+$Comp
+L EKR82-rescue:HOLE-EKR82-cache THLogo1
+U 1 1 60C38EB6
+P 2125 6075
+F 0 "THLogo1" H 2125 6075 60  0000 C CNN
+F 1 "HOLE" H 2125 5975 60  0000 C CNN
+F 2 "EKR82-footprint:EKR82-2" H 2125 6075 60  0001 C CNN
+F 3 "" H 2125 6075 60  0000 C CNN
+	1    2125 6075
+	1    0    0    -1
+$EndComp
+$Comp
+L EKR82-rescue:HOLE-EKR82-cache THLogo2
+U 1 1 60C8CADE
+P 2875 6025
+F 0 "THLogo2" H 2875 6025 60  0000 C CNN
+F 1 "HOLE" H 2875 5925 60  0000 C CNN
+F 2 "Symbol:OSHW-Symbol_8.9x8mm_SilkScreen" H 2875 6025 60  0001 C CNN
+F 3 "" H 2875 6025 60  0000 C CNN
+	1    2875 6025
+	1    0    0    -1
+$EndComp
+$Comp
+L EKR82-rescue:HOLE-EKR82-cache THLogo3
+U 1 1 60CA1C7A
+P 3525 6225
+F 0 "THLogo3" H 3525 6225 60  0000 C CNN
+F 1 "HOLE" H 3525 6125 60  0000 C CNN
+F 2 "Symbol:OSHW-Symbol_8.9x8mm_SilkScreen" H 3525 6225 60  0001 C CNN
+F 3 "" H 3525 6225 60  0000 C CNN
+	1    3525 6225
+	1    0    0    -1
+$EndComp
 $EndSCHEMATC

Commit message: change arduino footprint and move
Parts:
- U1: footprint EKR82-footprint:ProMicro_rev2 -> EKR82-footprint:ProMicro_rev
Changed lines of the file:
@@
 F 0 "U1" H 3200 3350 60  0000 C CNN
 F 1 "ProMicro" H 3200 1950 60  0000 C CNN
-F 2 "EKR82-footprint:ProMicro_rev2" H 3300 1600 60  0001 C CNN
+F 2 "EKR82-footprint:ProMicro_rev" H 3300 1600 60  0001 C CNN
 F 3 "" H 3300 1600 60  0000 C CNN
 	1    3200 2650
